File: host.kicad_sch (KiCad schematic)
At the start: 5 parts, among them J1 USB_C_Receptacle

Commit message: Used steppenprobe as base for our UART and JTAG.
Connections:
- net DN_HOST renamed DM_H
- net DP_HOST renamed DP_H
Changed lines of the file:
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@@
 		)
 	)
-	(global_label "DP_HOST"
+	(hierarchical_label "DP_H"
 		(shape input)
 		(at 52.07 44.45 0)
@@
 			(justify left)
 		)
-		(property "Intersheetrefs" "${INTERSHEET_REFS}"
-			(at 63.4009 44.45 0)
-			(effects
-				(font
-					(size 1.27 1.27)
-				)
-				(justify left)
-				(hide yes)
-			)
-		)
 	)
-	(global_label "DN_HOST"
+	(hierarchical_label "DM_H"
 		(shape input)
 		(at 67.31 39.37 0)
@@
 			(justify left)
 		)
-		(property "Intersheetrefs" "${INTERSHEET_REFS}"
-			(at 78.7014 39.37 0)
-			(effects
-				(font
-					(size 1.27 1.27)
-				)
-				(justify left)
-				(hide yes)
-			)
-		)
 	)
-	(global_label "VBUS"
+	(hierarchical_label "VBUS"
 		(shape input)
 		(at 92.71 25.4 0)
@@
 			(justify left)
 		)
-		(property "Intersheetrefs" "${INTERSHEET_REFS}"
-			(at 100.5938 25.4 0)
-			(effects
-				(font
-					(size 1.27 1.27)
-				)
-				(justify left)
-				(hide yes)
-			)
-		)
 	)

Commit message: started pcb layout, host and usbhub done
Parts:
- removed F1: Polyfuse, symbol Device:Polyfuse
- J1: footprint (none) -> Connector_USB:USB_C_Receptacle_HRO_TYPE-C-31-M-12
- R1, R2: footprint (none) -> Resistor_SMD:R_0603_1608Metric
Connections:
- net VBUS: now also J1.A4 (VBUS), J1.A9 (VBUS), J1.B4 (VBUS), J1.B9 (VBUS)
Changed lines of the file:
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@@
 	(wire
 		(pts
-			(xy 60.96 31.75) (xy 60.96 33.02)
+			(xy 67.31 31.75) (xy 67.31 33.02)
 		)
 		(stroke
@@
 	(wire
 		(pts
+			(xy 41.91 25.4) (xy 87.63 25.4)
+		)
+		(stroke
+			(width 0)
+			(type default)
+		)
+	)
+	(wire
+		(pts
 			(xy 41.91 39.37) (xy 66.04 39.37)
 		)
@@
 	(wire
 		(pts
-			(xy 49.53 25.4) (xy 87.63 25.4)
-		)
-		(stroke
-			(width 0)
-			(type default)
-		)
-	)
-	(wire
-		(pts
 			(xy 87.63 68.58) (xy 78.74 68.58)
 		)
@@
 	(wire
 		(pts
-			(xy 66.04 39.37) (xy 67.31 39.37)
+			(xy 66.04 39.37) (xy 71.12 39.37)
 		)
 		(stroke
@@
 	(wire
 		(pts
-			(xy 60.96 31.75) (xy 58.42 31.75)
+			(xy 67.31 31.75) (xy 58.42 31.75)
 		)
 		(stroke
@@
 	(hierarchical_label "DM_H"
 		(shape input)
-		(at 67.31 39.37 0)
+		(at 71.12 39.37 0)
 		(fields_autoplaced yes)
 		(effects
@@
 	)
 	(symbol
-		(lib_id "Device:Polyfuse")
-		(at 45.72 25.4 90)
+		(lib_id "power:GND")
+		(at 67.31 33.02 0)
 		(unit 1)
 		(exclude_from_sim no)
@@
 		(dnp no)
 		(fields_autoplaced yes)
-		(property "Reference" "F1"
-			(at 45.72 19.05 90)
-			(effects
-				(font
-					(size 1.27 1.27)
-				)
-			)
-		)
-		(property "Value" "Polyfuse"
-			(at 45.72 21.59 90)
+		(property "Reference" "#PWR02"
+			(at 67.31 39.37 0)
+			(effects
+				(font
+					(size 1.27 1.27)
+				)
+				(hide yes)
+			)
+		)
+		(property "Value" "GND"
+			(at 67.31 38.1 0)
 			(effects
 				(font
@@
 		)
 		(property "Footprint" ""
-			(at 50.8 24.13 0)
-			(effects
-				(font
-					(size 1.27 1.27)
-				)
-				(justify left)
-				(hide yes)
-			)
-		)
-		(property "Datasheet" "~"
-			(at 45.72 25.4 0)
-			(effects
-				(font
-					(size 1.27 1.27)
-				)
-				(hide yes)
-			)
-		)
-		(property "Description" "Resettable fuse, polymeric positive temperature coefficient"
-			(at 45.72 25.4 0)
+			(at 67.31 33.02 0)
+			(effects
+				(font
+					(size 1.27 1.27)
+				)
+				(hide yes)
+			)
+		)
+		(property "Datasheet" ""
+			(at 67.31 33.02 0)
+			(effects
+				(font
+					(size 1.27 1.27)
+				)
+				(hide yes)
+			)
+		)
+		(property "Description" "Power symbol creates a global label with name \"GND\" , ground"
+			(at 67.31 33.02 0)
 			(effects
 				(font
@@
 		(pin "1"
 		)
-		(pin "2"
-		)
 		(instances
-			(project "debug_board"
+			(project ""
 				(path "/9ba02813-5189-4482-9c9e-35a29bc7aded/3b80f853-6f7e-43fb-bbcc-e9ff1b9e9a11"
-					(reference "F1")
+					(reference "#PWR02")
 					(unit 1)
 				)
@@
 			)
 		)
-		(property "Footprint" ""
+		(property "Footprint" "Connector_USB:USB_C_Receptacle_HRO_TYPE-C-31-M-12"
 			(at 30.48 50.8 0)
 			(effects
@@
 			)
 		)
-		(property "Footprint" ""
+		(property "Footprint" "Resistor_SMD:R_0603_1608Metric"
 			(at 54.864 32.004 90)
 			(effects
@@
 				(path "/9ba02813-5189-4482-9c9e-35a29bc7aded/3b80f853-6f7e-43fb-bbcc-e9ff1b9e9a11"
 					(reference "R2")
-					(unit 1)
-				)
-			)
-		)
-	)
-	(symbol
-		(lib_id "power:GND")
-		(at 60.96 33.02 0)
-		(unit 1)
-		(exclude_from_sim no)
-		(in_bom yes)
-		(on_board yes)
-		(dnp no)
-		(fields_autoplaced yes)
-		(property "Reference" "#PWR02"
-			(at 60.96 39.37 0)
-			(effects
-				(font
-					(size 1.27 1.27)
-				)
-				(hide yes)
-			)
-		)
-		(property "Value" "GND"
-			(at 60.96 38.1 0)
-			(effects
-				(font
-					(size 1.27 1.27)
-				)
-			)
-		)
-		(property "Footprint" ""
-			(at 60.96 33.02 0)
-			(effects
-				(font
-					(size 1.27 1.27)
-				)
-				(hide yes)
-			)
-		)
-		(property "Datasheet" ""
-			(at 60.96 33.02 0)
-			(effects
-				(font
-					(size 1.27 1.27)
-				)
-				(hide yes)
-			)
-		)
-		(property "Description" "Power symbol creates a global label with name \"GND\" , ground"
-			(at 60.96 33.02 0)
-			(effects
-				(font
-					(size 1.27 1.27)
-				)
-				(hide yes)
-			)
-		)
-		(pin "1"
-		)
-		(instances
-			(project "debug_board"
-				(path "/9ba02813-5189-4482-9c9e-35a29bc7aded/3b80f853-6f7e-43fb-bbcc-e9ff1b9e9a11"
-					(reference "#PWR02")
 					(unit 1)
 				)
@@
 			)
 		)
-		(property "Footprint" ""
+		(property "Footprint" "Resistor_SMD:R_0603_1608Metric"
 			(at 54.864 29.464 90)
 			(effects
