File: debug_board.kicad_pcb (KiCad board)
At the start: 2 copper layers, 16.9 x 6.4 mm, 136 parts, among them IC1 TCAN3413DRBR, IC10 LMS1585AISX-3.3_NO, IC3 CYPD3177-24LQXQ, IC4 DMP3013SFV-7, IC5 DMP3013SFV-7, IC6 DMP3013SFV-7, IC7 DMP3013SFV-7, IC8 MAX77857CEWB+T, IC9 TPS73616DBVR, J1 USB_C_Receptacle, J2 USB_C_Receptacle_PowerOnly_24P, J3 Conn_01x02_Pin, J4 Conn_02x13_Row_Letter_Last, Q1 2N7002, SW1 SW_SPDT, SW2 SW_Push, SW3 SW_SPDT, SW4 SW_Push, U1 STM32F072RBH6, U10 74LVC1G125, U11 74LVC1G125, U12 74LVC1G125, U13 74LVC1G125, U2 USB2514B_Bi, U4 93LCxxB, U5 FT2232HL, U6 74LVC1G125, U7 74LVC1G126, U8 74LVC1G125, U9 74LVC1G125, Y1 ABLS-24.000MHZ-B4-T, Y2 Crystal_GND24

Commit message: routed stm32
Parts:
- removed C41, C42: 100nf, Capacitor_SMD:C_0603_1608Metric
- removed D7: LED, LED_SMD:LED_0603_1608Metric
- removed R17: 330, Resistor_SMD:R_0603_1608Metric
- removed Y1: ABLS-24.000MHZ-B4-T, SamacSys_Parts:ABLS24000MHZB4T
- added C50: 4.7uF, Capacitor_SMD:C_0603_1608Metric, F.Cu at (49.0, 100.6)
- added C51: 4.7uF, Capacitor_SMD:C_0603_1608Metric, F.Cu at (57.7, 103.2)
- added C52: 1uF, Capacitor_SMD:C_0603_1608Metric, F.Cu at (49.2, 87.5)
- added Y3: ABM3B-24.000MHZ-B2-T, SamacSys_Parts:ABM3B, F.Cu at (34.7, 52.7)
- SW3: value SW_SPDT -> SW_Push; footprint Button_Switch_SMD:SW_SPDT_PCM12 -> Button_Switch_SMD:SW_Push_1P1T_XKB_TS-1187A
- U1: footprint Package_BGA:UFBGA-64_5x5mm_Layout8x8_P0.5mm -> Package_QFP:LQFP-64_10x10mm_P0.5mm
- moved J4 195.1 mm to (151.4, 90.4)
- moved C19 132.5 mm to (57.7, 101.8), turned to 180 degrees
- moved C39 131.4 mm to (61.8, 99.8), turned to 90 degrees
- moved C43 128.3 mm to (55.0, 103.0), turned to 90 degrees
- moved C40 124.6 mm to (62.5, 89.3)
- moved C38 122.5 mm to (49.0, 99.1), turned to 180 degrees
- moved C4 119.6 mm to (50.8, 87.5), turned to 90 degrees
- moved SW4 118.2 mm to (51.4, 105.3), turned to 90 degrees
- moved R9 115.0 mm to (46.0, 95.7)
- moved IC1 110.9 mm to (44.4, 98.3), turned to 180 degrees
- moved R15 110.1 mm to (40.7, 96.8)
- moved U1 109.9 mm to (55.8, 94.2), turned to 90 degrees
- moved SW3 104.6 mm to (38.8, 92.0), turned to 90 degrees
- moved C49 75.3 mm to (40.6, 41.8), turned to 90 degrees
- moved R38 73.0 mm to (38.9, 41.6), turned to 90 degrees
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Connections:
- IC3 pad 12: /Power/HPI_SDA -> unconnected-(IC3-HPI_SDA-Pad12)
- IC3 pad 13: /Power/HPI_SCL -> unconnected-(IC3-HPI_SCL-Pad13)
- R15 pad 1: Net-(U1-PB0) -> Net-(U1-PA14)
- R9 pad 2: Net-(U1-BOOT0) -> GND
- SW3 pad 1: GND -> +3.3V
Routing:
- net +3.3V: track 9.47 -> 41.6 mm
- net GND: track 11.3 -> 32.7 mm, vias 10 -> 11
- net /USB Hub/XIN: track 26.6 -> 11.4 mm
- net /USB Host/VBUS: track 16.0 -> 30.9 mm
- net Net-(R9-Pad1): track 0.00 -> 10.7 mm
- net /STM32/NRST: track 0.00 -> 10.2 mm
- net Net-(U2-RESET_N): track 0.00 -> 8.24 mm
- net /STM32/CAN TX: track 0.00 -> 5.20 mm
- net /USB Hub/XOUT: track 19.1 -> 14.1 mm
- net /STM32/CAN_RX: track 0.00 -> 4.60 mm
- net Net-(IC1-SHDNVIO): track 0.00 -> 1.67 mm
Other:
- board size 16.9 x 6.4 mm -> 16.8 x 6.4 mm

Commit message: pcb routed!!!!!!!
Parts:
- removed C11, C12: 10uF 25V, Capacitor_SMD:C_0603_1608Metric
- removed C13, C14: 22uF 25V, Capacitor_SMD:C_0603_1608Metric
- removed C15: 2.2uF 10V, Capacitor_SMD:C_0603_1608Metric
- removed C16, C17: 0.22uF 25V, Capacitor_SMD:C_0603_1608Metric
- removed C18: 0.47uF 6.3V, Capacitor_SMD:C_0603_1608Metric
- removed C35, C36, C37: 100nF, Capacitor_SMD:C_0603_1608Metric
- removed FB2, FB3: Ferrite_Bead, Inductor_SMD:L_0603_1608Metric
- removed IC8: MAX77857CEWB+T, SamacSys_Parts:BGA35C40P7X5_283X203X69
- removed IC9: TPS73616DBVR, SamacSys_Parts:SOT95P280X145-5N
- removed J4: Conn_02x13_Row_Letter_Last, Connector_Samtec_HSEC8:Samtec_HSEC8-113-X-X-DV_2x13_P0.8mm_Wing_Edge
- removed L1: 1.5uH, Inductor_SMD:L_0805_2012Metric
- removed Q1: 2N7002, Package_TO_SOT_SMD:SOT-23
- removed R26, R27, R29, R30: 10k, Resistor_SMD:R_0603_1608Metric
- removed R28: 100k, Resistor_SMD:R_0603_1608Metric
- removed SW1: SW_SPDT, Button_Switch_SMD:SW_SPDT_PCM12
- removed SW2: SW_Push, Button_Switch_SMD:SW_Push_1P1T_XKB_TS-1187A
- removed U10, U11, U12, U13, U6, U8, U9: 74LVC1G125, Package_TO_SOT_SMD:SOT-353_SC-70-5
- removed U7: 74LVC1G126, Package_TO_SOT_SMD:SOT-353_SC-70-5
- added IC2: TLV74018PDBVR, SamacSys_Parts:SOT95P280X145-5N, F.Cu at (59.5, 71.0)
- C7: value 4.7nF -> 1uF
- C8: value 4.7nF -> 1nF
- J3: value Conn_01x02_Pin -> Conn_02x13_Row_Letter_Last; footprint TerminalBlock:TerminalBlock_Xinya_XY308-2.54-2P_1x02_P2.54mm_Horizontal -> Connector_Samtec_HSEC8:Samtec_HSEC8-113-X-X-DV_2x13_P0.8mm_Edge
- moved C32 179.7 mm to (89.7, 82.5), turned to -90 degrees
- moved C33 178.9 mm to (91.2, 77.8)
- moved C31 178.5 mm to (85.5, 87.7), turned to -90 degrees
- moved C21 176.4 mm to (84.5, 70.7), turned to 90 degrees
- moved C29 175.7 mm to (79.5, 89.8), turned to -90 degrees
- moved C25 175.2 mm to (86.0, 70.7), turned to 90 degrees
- moved R21 170.5 mm to (82.9, 92.8), turned to 90 degrees
- moved C5 169.1 mm to (78.2, 61.0)
- moved R33 168.6 mm to (79.2, 98.3), turned to 90 degrees
- moved C34 168.4 mm to (83.0, 70.7), turned to 90 degrees
- moved C28 168.1 mm to (74.0, 80.8), turned to 180 degrees
- moved R37 168.0 mm to (83.7, 98.3), turned to -90 degrees
- moved R36 167.8 mm to (82.2, 98.3), turned to 90 degrees
- moved R22 166.8 mm to (79.9, 92.8), turned to -90 degrees
- moved R34 166.1 mm to (77.8, 98.3), turned to 90 degrees
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Connections:
- C21 pad 1: +3V3 -> +3.3V
- C23 pad 1: /FTDI/VPLL -> +3.3V
- C24 pad 1: /FTDI/VPHY -> +3.3V
- C26 pad 1: /FTDI/VPLL -> +3.3V
- C27 pad 1: /FTDI/VPHY -> +3.3V
- C29 pad 1: +3V3 -> +3.3V
- C31 pad 1: +3V3 -> +3.3V
- C33 pad 1: +3V3 -> +3.3V
- C34 pad 1: +3V3 -> +3.3V
- C5 pad 1: +3V3 -> +3.3V
- D10 pad 2: +3V3 -> +3.3V
- D11 pad 2: +3V3 -> +3.3V
- D12 pad 2: +3V3 -> +3.3V
- D5 pad 3: /Power/VOUT -> +5V
- D6 pad 3: /Power/VOUT -> +5V
- D9 pad 2: +3V3 -> +3.3V
- IC10 pad 5: (no net) -> +3.3V
- IC10 pad 6: (no net) -> +3.3V
- IC3 pad 19: Net-(IC3-GND_1) -> GND
- IC3 pad 22: Net-(IC3-GND_1) -> GND
- IC3 pad 25: unconnected-(IC3-GND_3-Pad25) -> GND
- J3 pad 1: /Power/VOUT -> +3.3V
- R20 pad 2: +3V3 -> +3.3V
- R31 pad 1: /FTDI/SRST -> /FTDI/SRST_N_TRGT
- R31 pad 2: /FTDI/SRST_N_R -> /FTDI/SRST
- R32 pad 1: /FTDI/TCK -> /FTDI/TCK_TRGT
- R32 pad 2: /FTDI/TCK_R -> /FTDI/TCK
- R33 pad 1: /FTDI/TMS -> /FTDI/TMS_TRGT
- R33 pad 2: /FTDI/TMS_R -> /FTDI/TMS
- R34 pad 1: /FTDI/TDO -> /FTDI/TDO_TRGT
- R34 pad 2: /FTDI/TDO_R -> /FTDI/TDO
- R35 pad 1: /FTDI/TDI -> /FTDI/TDI_TRGT
- R35 pad 2: /FTDI/TDI_R -> /FTDI/TDI
- R36 pad 1: /FTDI/TXD -> /FTDI/TXD_TRGT
- R36 pad 2: /FTDI/TXD_R -> /FTDI/TXD
- R37 pad 1: /FTDI/RXD_R -> /FTDI/RXD
- R37 pad 2: /FTDI/RXD -> /FTDI/RXD_TRGT
- U2 pad 1: /FTDI/DM -> /STM32/USB-
- U2 pad 2: /FTDI/DP -> /STM32/USB+
- U2 pad 6: /Connector/USB2-? -> /FTDI/DM
- U2 pad 7: /Connector/USB2+? -> /FTDI/DP
- U2 pad 8: /STM32/USB- -> /Connector/USB2-?
- U2 pad 9: /STM32/USB+ -> /Connector/USB2+?
- U4 pad 8: +3V3 -> +3.3V
- U5 pad 20: +3V3 -> +3.3V
- U5 pad 31: +3V3 -> +3.3V
- U5 pad 4: /FTDI/VPHY -> +3.3V
- U5 pad 42: +3V3 -> +3.3V
- U5 pad 50: +3V3 -> +3.3V
- U5 pad 56: +3V3 -> +3.3V
- U5 pad 9: /FTDI/VPLL -> +3.3V
Routing:
- net +3.3V: track 41.6 -> 359.7 mm, vias 0 -> 26
- net GND: track 32.7 -> 126.9 mm, vias 11 -> 58
- net +5V: track 0.00 -> 82.6 mm, vias 0 -> 16
- net /Power/VBUS: track 0.00 -> 69.6 mm, vias 0 -> 22
- net +1V8: track 0.00 -> 59.3 mm, vias 0 -> 5
- net /Power/SAFE_PWR: track 0.00 -> 52.7 mm
- net /Connector/USB-: track 0.00 -> 48.6 mm, vias 0 -> 1
- net /Connector/USB+: track 0.00 -> 47.5 mm, vias 0 -> 1
- net /Connector/CANL: track 0.00 -> 47.0 mm, vias 0 -> 2
- net /Connector/CANH: track 0.00 -> 46.8 mm, vias 0 -> 2
- net /Connector/USB2-?: track 0.00 -> 42.6 mm, vias 0 -> 3
- net /Connector/I2C_SDA: track 0.00 -> 42.6 mm, vias 0 -> 3
- net /Connector/USB2+?: track 0.00 -> 42.1 mm, vias 0 -> 3
- net /Connector/I2C_SCL: track 0.00 -> 41.4 mm, vias 0 -> 3
- net /Power/VBUS_FET: track 0.00 -> 40.9 mm
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- added copper zone on B.Cu, net +3.3V
- added copper zone on F.Cu, net +3.3V
- added copper zone on B.Cu, net +5V
- added copper zone on F.Cu, net +5V
- added copper zone on B.Cu, net /Power/VBUS
- added copper zone on F.Cu, net /Power/VBUS
- added copper zone on F.Cu, net /Power/VDC_OUT
- added copper zone on F.Cu, net /Power/VOUT_PD
- added copper zone on B.Cu, net GND
- added copper zone on F.Cu, net Net-(D4-K)
- added copper zone on F.Cu, net Net-(IC6-D_1)
Other:
- board size 16.8 x 6.4 mm -> 68.4 x 76 mm
- board text added: "SAFE MODE"
