File: debug_board.kicad_sch (KiCad schematic)
At the start: 0 parts

Commit message: routed stm32
Other:
- sheet Power ports: added HPI_SCL, HPI_SDA; removed none
Changed lines of the file:
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@@
+			)
+		)
+		(pin "HPI_SCL" input
+			(at 35.56 88.9 270)
+			(effects
+				(font
+					(size 1.27 1.27)
+				)
+				(justify left)
+			)
+		)
+		(pin "HPI_SDA" input
+			(at 39.37 88.9 270)
+			(effects
+				(font
+					(size 1.27 1.27)
+				)
+				(justify left)
 			)
 		)

Commit message: pcb routed!!!!!!!
Other:
- sheet FTDI ports: added RXD_TRGT, SRST_TRGT, TCK_TRGT, TDI_TRGT, TDO_TRGT, TMS_TRGT, TXD_TRGT; removed RXD, SRST, TCK, TDI, TDO, TMS, TXD
Changed lines of the file:
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@@
 			)
 		)
-		(pin "SRST" input
+		(pin "TMS_TRGT" input
+			(at 114.3 46.99 0)
+			(effects
+				(font
+					(size 1.27 1.27)
+				)
+				(justify right)
+			)
+		)
+		(pin "SRST_TRGT" input
 			(at 114.3 41.91 0)
 			(effects
@@
 			)
 		)
-		(pin "TCK" input
+		(pin "TDI_TRGT" input
+			(at 114.3 52.07 0)
+			(effects
+				(font
+					(size 1.27 1.27)
+				)
+				(justify right)
+			)
+		)
+		(pin "TDO_TRGT" input
+			(at 114.3 49.53 0)
+			(effects
+				(font
+					(size 1.27 1.27)
+				)
+				(justify right)
+			)
+		)
+		(pin "TXD_TRGT" input
+			(at 114.3 54.61 0)
+			(effects
+				(font
+					(size 1.27 1.27)
+				)
+				(justify right)
+			)
+		)
+		(pin "TCK_TRGT" input
 			(at 114.3 44.45 0)
 			(effects
@@
 			)
 		)
-		(pin "TMS" input
-			(at 114.3 46.99 0)
-			(effects
-				(font
-					(size 1.27 1.27)
-				)
-				(justify right)
-			)
-		)
-		(pin "TDO" input
-			(at 114.3 49.53 0)
-			(effects
-				(font
-					(size 1.27 1.27)
-				)
-				(justify right)
-			)
-		)
-		(pin "TDI" input
-			(at 114.3 52.07 0)
-			(effects
-				(font
-					(size 1.27 1.27)
-				)
-				(justify right)
-			)
-		)
-		(pin "TXD" input
-			(at 114.3 54.61 0)
-			(effects
-				(font
-					(size 1.27 1.27)
-				)
-				(justify right)
-			)
-		)
-		(pin "RXD" input
+		(pin "RXD_TRGT" input
 			(at 114.3 57.15 0)
 			(effects
