File: power.kicad_sch (KiCad schematic)
At the start: 37 parts, among them IC10 LMS1585AISX-3.3_NO, IC3 CYPD3177-24LQXQ, IC4 DMP3013SFV-7, IC5 DMP3013SFV-7, IC6 DMP3013SFV-7, IC7 DMP3013SFV-7, IC8 MAX77857CEWB+T, IC9 TPS73616DBVR, J2 USB_C_Receptacle_PowerOnly_24P, J3 Conn_01x02_Pin

Commit message: started pcb layout, host and usbhub done
Parts:
- C10, C11, C12, C13, C14, C15, C16, C17, C18, C3, C6, C7, C8: footprint (none) -> Capacitor_SMD:C_0603_1608Metric
- C9: value 3.3uF -> 3.3uF,15V; footprint (none) -> Capacitor_SMD:C_0603_1608Metric
- D2: footprint (none) -> LED_SMD:LED_0603_1608Metric
- D3: footprint (none) -> Diode_SMD:D_SOD-323_HandSoldering
- D4: footprint (none) -> SODFL2513X100N
- J2: footprint (none) -> Connector_USB:USB_C_Receptacle_GCT_USB4135-GF-A_6P_TopMnt_Horizontal
- J3: footprint (none) -> TerminalBlock:TerminalBlock_Xinya_XY308-2.54-2P_1x02_P2.54mm_Horizontal
- L1: footprint (none) -> Inductor_SMD:L_0805_2012Metric
- R10, R11, R12, R13, R14, R3, R4: footprint (none) -> Resistor_SMD:R_0603_1608Metric
Connections:
- net +3.3V: no longer C11.2, C12.2, C13.2, C14.2, C15.2, C18.2, C3.2, C6.2, C7.2, C8.2, C9.2, D3.2 (A), IC10.1 (ADJ/GND), IC3.1 (VBUS_MIN), IC3.2 (VBUS_MAX), IC3.6 (ISNK_FINE), IC8.C3 (PGND_1), IC8.C4 (PGND_2), IC8.C5 (PGND_3), IC8.C6 (PGND_4), IC8.C7 (PGND_5), IC8.D2 (PGND_6), IC8.D3 (PGND_7), IC8.E2 (AGND), IC9.2 (GND), J2.A1 (GND), J2.A12 (GND), J2.B1 (GND), J2.B12 (GND), J2.S1 (SHIELD), J3.2 (Pin_2), R3.2
- new net GND: C11.2, C12.2, C13.2, C14.2, C15.2, C18.2, C3.2, C6.2, C7.2, C8.2, C9.2, D3.2 (A), IC10.1 (ADJ/GND), IC3.1 (VBUS_MIN), IC3.2 (VBUS_MAX), IC3.6 (ISNK_FINE), IC8.C3 (PGND_1), IC8.C4 (PGND_2), IC8.C5 (PGND_3), IC8.C6 (PGND_4), IC8.C7 (PGND_5), IC8.D2 (PGND_6), IC8.D3 (PGND_7), IC8.E2 (AGND), IC9.2 (GND), J2.A1 (GND), J2.A12 (GND), J2.B1 (GND), J2.B12 (GND), J2.S1 (SHIELD), J3.2 (Pin_2), R3.2
Changed lines of the file:
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@@
 	(paper "A3")
 	(junction
-		(at 67.31 39.37)
-		(diameter 0)
-		(color 0 0 0 0)
-	)
-	(junction
 		(at 201.93 99.06)
 		(diameter 0)
@@
 	)
 	(junction
-		(at 67.31 34.29)
-		(diameter 0)
-		(color 0 0 0 0)
-	)
-	(junction
 		(at 153.67 30.48)
 		(diameter 0)
@@
 	(wire
 		(pts
-			(xy 67.31 34.29) (xy 67.31 39.37)
-		)
-		(stroke
-			(width 0)
-			(type default)
-		)
-	)
-	(wire
-		(pts
 			(xy 66.04 200.66) (xy 66.04 203.2)
 		)
@@
 			)
 		)
-		(property "Footprint" ""
+		(property "Footprint" "Resistor_SMD:R_0603_1608Metric"
 			(at 202.946 95.504 90)
 			(effects
@@
 			)
 		)
-		(property "Footprint" ""
+		(property "Footprint" "SODFL2513X100N"
 			(at 198.12 95.25 0)
 			(effects
@@
 			)
 		)
-		(property "Value" "3.3uF"
+		(property "Value" "3.3uF,15V"
 			(at 53.086 59.182 0)
 			(effects
@@
 			)
 		)
-		(property "Footprint" ""
+		(property "Footprint" "Capacitor_SMD:C_0603_1608Metric"
 			(at 55.88 63.5 0)
 			(effects
@@
 			)
 		)
-		(property "Footprint" ""
+		(property "Footprint" "Capacitor_SMD:C_0603_1608Metric"
 			(at 60.96 189.23 0)
 			(effects
@@
 			)
 		)
-		(property "Footprint" ""
+		(property "Footprint" "Capacitor_SMD:C_0603_1608Metric"
 			(at 116.84 214.63 0)
 			(effects
@@
 			)
 		)
-		(property "Footprint" ""
+		(property "Footprint" "Connector_USB:USB_C_Receptacle_GCT_USB4135-GF-A_6P_TopMnt_Horizontal"
 			(at 38.1 66.04 0)
 			(effects
@@
 			)
 		)
-		(property "Footprint" ""
+		(property "Footprint" "Capacitor_SMD:C_0603_1608Metric"
 			(at 125.73 185.42 0)
 			(effects
@@
 			)
 		)
-		(property "Footprint" ""
+		(property "Footprint" "Inductor_SMD:L_0805_2012Metric"
 			(at 135.89 182.88 0)
 			(effects
@@
 			)
 		)
-		(property "Footprint" ""
+		(property "Footprint" "Resistor_SMD:R_0603_1608Metric"
 			(at 154.686 35.814 90)
 			(effects
@@
 			)
 		)
-		(property "Footprint" ""
+		(property "Footprint" "LED_SMD:LED_0603_1608Metric"
 			(at 81.28 102.87 0)
 			(effects
@@
 			)
 		)
-		(property "Footprint" ""
+		(property "Footprint" "Capacitor_SMD:C_0603_1608Metric"
 			(at 127 214.63 0)
 			(effects
@@
 			)
 		)
-		(property "Footprint" ""
+		(property "Footprint" "Resistor_SMD:R_0603_1608Metric"
 			(at 79.756 110.744 90)
 			(effects
@@
 			)
 		)
-		(property "Footprint" ""
+		(property "Footprint" "Capacitor_SMD:C_0603_1608Metric"
 			(at 146.05 185.42 0)
 			(effects
@@
 			)
 		)
-		(property "Footprint" ""
+		(property "Footprint" "Resistor_SMD:R_0603_1608Metric"
 			(at 103.124 72.644 90)
 			(effects
@@
 			)
 		)
-		(property "Footprint" ""
+		(property "Footprint" "Capacitor_SMD:C_0603_1608Metric"
 			(at 148.2852 101.6 0)
 			(effects
@@
 			)
 		)
-		(property "Footprint" ""
+		(property "Footprint" "TerminalBlock:TerminalBlock_Xinya_XY308-2.54-2P_1x02_P2.54mm_Horizontal"
 			(at 62.23 130.81 0)
 			(effects
@@
 			)
 		)
-		(property "Footprint" ""
+		(property "Footprint" "Resistor_SMD:R_0603_1608Metric"
 			(at 103.124 70.104 90)
 			(effects
@@
 			)
 		)
-		(property "Footprint" ""
+		(property "Footprint" "Capacitor_SMD:C_0603_1608Metric"
 			(at 73.66 36.83 0)
 			(effects
@@
 			)
 		)
-		(property "Footprint" ""
+		(property "Footprint" "Capacitor_SMD:C_0603_1608Metric"
 			(at 49.53 213.36 0)
 			(effects
@@
 			)
 		)
-		(property "Footprint" ""
+		(property "Footprint" "Resistor_SMD:R_0603_1608Metric"
 			(at 82.296 110.744 90)
 			(effects
@@
 			)
 		)
-		(property "Footprint" ""
+		(property "Footprint" "Capacitor_SMD:C_0603_1608Metric"
 			(at 77.47 36.83 0)
 			(effects
@@
 			)
 		)
-		(property "Footprint" ""
+		(property "Footprint" "Capacitor_SMD:C_0603_1608Metric"
 			(at 69.85 36.83 0)
 			(effects
@@
 			)
 		)
-		(property "Footprint" ""
+		(property "Footprint" "Capacitor_SMD:C_0603_1608Metric"
 			(at 35.56 180.34 0)
 			(effects
@@
 			)
 		)
-		(property "Footprint" ""
+		(property "Footprint" "Resistor_SMD:R_0603_1608Metric"
 			(at 159.766 98.044 90)
 			(effects
@@
 			)
 		)
-		(property "Footprint" ""
+		(property "Footprint" "Capacitor_SMD:C_0603_1608Metric"
 			(at 80.01 25.4 0)
 			(effects
@@
 			)
 		)
-		(property "Footprint" ""
+		(property "Footprint" "Diode_SMD:D_SOD-323_HandSoldering"
 			(at 49.53 64.77 0)
 			(effects
@@
 			)
 		)
-		(property "Footprint" ""
+		(property "Footprint" "Capacitor_SMD:C_0603_1608Metric"
 			(at 50.8 189.23 0)
 			(effects

Commit message: routed stm32
Connections:
- net HPI_SCL: no longer names the net of IC3.13 (HPI_SCL)
- net HPI_SDA: no longer names the net of IC3.12 (HPI_SDA)
- no-connect marks 10 -> 14
Changed lines of the file:
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@@
+	)
+	(no_connect
+		(at 58.42 78.74)
 	)
 	(no_connect
@@
 	)
 	(no_connect
+		(at 25.4 252.73)
+	)
+	(no_connect
+		(at 73.66 99.06)
+	)
+	(no_connect
 		(at 58.42 71.12)
 	)
@@
 	(no_connect
 		(at 124.46 140.97)
+	)
+	(no_connect
+		(at 35.56 259.08)
 	)
 	(no_connect
@@
 		)
 	)
-	(hierarchical_label "HPI_SCL"
-		(shape input)
-		(at 58.42 78.74 180)
-		(fields_autoplaced yes)
-		(effects
-			(font
-				(size 1.27 1.27)
-			)
-			(justify right)
-		)
-	)
-	(hierarchical_label "HPI_SDA"
-		(shape input)
-		(at 73.66 99.06 270)
-		(fields_autoplaced yes)
-		(effects
-			(font
-				(size 1.27 1.27)
-			)
-			(justify right)
-		)
-	)

Commit message: pcb routed!!!!!!!
Parts:
- removed C11, C12: 10uF 25V, Capacitor_SMD:C_0603_1608Metric, symbol Device:C_Small
- removed C13, C14: 22uF 25V, Capacitor_SMD:C_0603_1608Metric, symbol Device:C_Small
- removed C15: 2.2uF 10V, Capacitor_SMD:C_0603_1608Metric, symbol Device:C_Small
- removed C16, C17: 0.22uF 25V, Capacitor_SMD:C_0603_1608Metric, symbol Device:C_Small
- removed C18: 0.47uF 6.3V, Capacitor_SMD:C_0603_1608Metric, symbol Device:C_Small
- removed IC8: MAX77857CEWB+T, BGA35C40P7X5_283X203X69, symbol SamacSys_Parts:MAX77857CEWB+T
- removed IC9: TPS73616DBVR, SOT95P280X145-5N, symbol SamacSys_Parts:TPS73616DBVR
- removed J3: Conn_01x02_Pin, TerminalBlock:TerminalBlock_Xinya_XY308-2.54-2P_1x02_P2.54mm_Horizontal, symbol Connector:Conn_01x02_Pin
- removed L1: 1.5uH, Inductor_SMD:L_0805_2012Metric, symbol Device:L
- added IC2: TLV74018PDBVR, SOT95P280X145-5N, symbol SamacSys_Parts:TLV74018PDBVR
- C7: value 4.7nF -> 1uF
- C8: value 4.7nF -> 1nF
Connections:
- net VOUT is gone; now on net +5V: D5.3 (K), D6.3 (K)
- net +1V8: now also IC2.5 (OUT)
- net +3.3V: now also IC10.5 (VOUT), IC10.6 (VOUT)
- net +5V: now also IC2.1 (IN), IC2.3 (EN)
- net GND: now also IC3.19 (GND_1), IC3.22 (GND_2), IC3.25 (GND_3), IC2.2 (GND)
- no-connect marks 14 -> 10
Other:
- note removed: "STABILZE USB INPUT TO 5V"
- note removed: "VOUT TO 1.8"
